File: v3/hydrogen.brd (EAGLE design)
At the start: 33 x 27.9 mm, 19 parts, among them U1 TPS61088VQFN20

Commit message: Hydrogen board v1r0 off to OSH park.
Parts:
- added H: 1, 32bits:PERIODIC_SYMBOL_BACK
- moved R1 0.63 mm to (30.5, 5.71)
Connections:
- net GND: now also U1.P$25
Routing:
- net LED_ANODE: track 3.38 -> 2.74 mm
- added copper zone on layer 16, net GND
Other:
- board text added: "3.0-4.2v"
- board text added: "6v"
Changed lines of the file:
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@@
 <wire x1="24.13" y1="6.0325" x2="24.13" y2="1.5875" width="0.27" layer="25"/>
 <wire x1="24.13" y1="1.5875" x2="23.495" y2="1.5875" width="0.27" layer="25"/>
+<text x="0.9525" y="20.955" size="0.8128" layer="21" font="vector">3.0-4.2v</text>
+<text x="26.035" y="6.6675" size="0.8128" layer="21" font="vector">6v</text>
 </plain>
 <attributes>
@@
 <attribute name="TOLERANCE" value="±5%" x="25.0825" y="17.4625" size="1.778" layer="27" rot="R270" display="off"/>
 <attribute name="OC_FARNELL" value="-" x="25.0825" y="17.4625" size="1.778" layer="27" rot="R270" display="off"/>
-<attribute name="NAME" x="24.9711" y="19.05" size="0.3048" layer="25" ratio="10" rot="SR90"/>
+<attribute name="NAME" x="24.9711" y="20.32" size="0.3048" layer="25" ratio="10" rot="SR90"/>
 </element>
 <element name="CCOMP2" library="Kemet_By_element14_Batch_1" package="CAPC1005X60N" value="36pF" x="23.495" y="17.4625" smashed="yes" rot="R270">
@@
 <attribute name="TOLERANCE" value="±5%" x="23.495" y="17.4625" size="1.778" layer="27" rot="R270" display="off"/>
 <attribute name="OC_FARNELL" value="1865427" x="23.495" y="17.4625" size="1.778" layer="27" rot="R270" display="off"/>
-<attribute name="NAME" x="23.4725" y="19.05" size="0.3048" layer="25" ratio="10" rot="SR90"/>
+<attribute name="NAME" x="23.4725" y="20.32" size="0.3048" layer="25" ratio="10" rot="SR90"/>
 </element>
 <element name="CIN" library="Kemet_By_element14_Batch_1" package="CAPC3216X180N" value="0.47uF" x="2.1925" y="10.2725" smashed="yes" rot="R90">
@@
 <attribute name="TOLERANCE" value="±1%" x="26.67" y="17.4625" size="1.778" layer="27" rot="R270" display="off"/>
 <attribute name="OC_FARNELL" value="1652743" x="26.67" y="17.4625" size="1.778" layer="27" rot="R270" display="off"/>
-<attribute name="NAME" x="26.6725" y="19.05" size="0.3048" layer="25" ratio="10" rot="SR90"/>
+<attribute name="NAME" x="26.6725" y="20.32" size="0.3048" layer="25" ratio="10" rot="SR90"/>
 </element>
 <element name="RFBT" library="Yageo_By_element14_Batch_1" package="RESC1608X60N" value="470K Ohms" x="26.6325" y="14.1025" smashed="yes" rot="R90">
@@
 <attribute name="TOLERANCE" value="±1%" x="22.225" y="17.4625" size="1.778" layer="27" rot="R90" display="off"/>
 <attribute name="OC_FARNELL" value="1150767" x="22.225" y="17.4625" size="1.778" layer="27" rot="R90" display="off"/>
-<attribute name="NAME" x="22.13" y="19.05" size="0.3048" layer="25" ratio="10" rot="SR90"/>
+<attribute name="NAME" x="22.13" y="20.32" size="0.3048" layer="25" ratio="10" rot="SR90"/>
 </element>
 <element name="RT" library="Vishay_By_element14_Batch_1" package="RESC1005X40N" value="261K Ohms" x="13.97" y="16.8275" smashed="yes" rot="R180">
@@
 <attribute name="OC_FARNELL" value="1179613" x="30.48" y="11.43" size="0.8128" layer="27" font="vector" rot="R270" display="off"/>
 <attribute name="OC_NEWARK" value="30K4956" x="30.48" y="11.43" size="0.8128" layer="27" font="vector" rot="R270" display="off"/>
-<attribute name="NAME" x="29.5656" y="14.0716" size="0.8128" layer="25" ratio="10" rot="SR0"/>
-</element>
-<element name="R1" library="Vishay_By_element14_Batch_1" package="RESC3216X71N" value="200 Ohms" x="30.48" y="5.08" smashed="yes" rot="R270">
-<attribute name="TOLERANCE" value="±5%" x="30.48" y="5.08" size="0.8128" layer="27" font="vector" rot="R270" display="off"/>
-<attribute name="WATTAGE" value="0.25W" x="30.48" y="5.08" size="0.8128" layer="27" font="vector" rot="R270" display="off"/>
-<attribute name="MPN" value="CRCW1206200RJNEA" x="30.48" y="5.08" size="0.8128" layer="27" font="vector" rot="R270" display="off"/>
-<attribute name="SUPPLIER" value="Vishay" x="30.48" y="5.08" size="0.8128" layer="27" font="vector" rot="R270" display="off"/>
-<attribute name="OC_FARNELL" value="1540005" x="30.48" y="5.08" size="0.8128" layer="27" font="vector" rot="R270" display="off"/>
-<attribute name="OC_NEWARK" value="59M6966" x="30.48" y="5.08" size="0.8128" layer="27" font="vector" rot="R270" display="off"/>
-<attribute name="NAME" x="31.1531" y="2.54" size="0.254" layer="25" ratio="10" rot="SR0"/>
+<attribute name="NAME" x="31.7881" y="11.5316" size="0.4064" layer="25" ratio="10" rot="SR0"/>
+</element>
+<element name="R1" library="Vishay_By_element14_Batch_1" package="RESC3216X71N" value="200 Ohms" x="30.48" y="5.715" smashed="yes" rot="R270">
+<attribute name="TOLERANCE" value="±5%" x="30.48" y="5.715" size="0.8128" layer="27" font="vector" rot="R270" display="off"/>
+<attribute name="WATTAGE" value="0.25W" x="30.48" y="5.715" size="0.8128" layer="27" font="vector" rot="R270" display="off"/>
+<attribute name="MPN" value="CRCW1206200RJNEA" x="30.48" y="5.715" size="0.8128" layer="27" font="vector" rot="R270" display="off"/>
+<attribute name="SUPPLIER" value="Vishay" x="30.48" y="5.715" size="0.8128" layer="27" font="vector" rot="R270" display="off"/>
+<attribute name="OC_FARNELL" value="1540005" x="30.48" y="5.715" size="0.8128" layer="27" font="vector" rot="R270" display="off"/>
+<attribute name="OC_NEWARK" value="59M6966" x="30.48" y="5.715" size="0.8128" layer="27" font="vector" rot="R270" display="off"/>
+<attribute name="NAME" x="31.1531" y="3.175" size="0.254" layer="25" ratio="10" rot="SR0"/>
+</element>
+<element name="H" library="32bits" package="PERIODIC_SYMBOL_BACK" value="1" x="1.905" y="11.43">
+<attribute name="DESC" value="rev.0" x="1.905" y="11.43" size="1.778" layer="27" display="off"/>
 </element>
 </elements>
@@
 <vertex x="0" y="27.94"/>
 <vertex x="0" y="0"/>
-<vertex x="33.02" y="0"/>
+<vertex x="22.86" y="0"/>
+<vertex x="22.86" y="11.43"/>
+<vertex x="33.02" y="11.43"/>
 <vertex x="33.02" y="27.94"/>
 </polygon>
@@
 <contactref element="J4" pad="2"/>
 <polygon width="0.27" layer="1" thermals="no">
-<vertex x="18.7325" y="16.1925"/>
-<vertex x="20.32" y="16.1925"/>
+<vertex x="18.7325" y="10.4775"/>
+<vertex x="20.32" y="10.4775"/>
+<vertex x="20.32" y="11.7475"/>
+<vertex x="21.59" y="11.7475"/>
+<vertex x="21.59" y="12.7"/>
+<vertex x="20.32" y="12.7"/>
 <vertex x="20.32" y="17.78"/>
 <vertex x="18.7325" y="17.78"/>
 </polygon>
 <contactref element="+6" pad="1"/>
+<contactref element="U1" pad="P$25"/>
+<polygon width="0.4064" layer="16">
+<vertex x="0" y="27.94"/>
+<vertex x="33.02" y="27.94"/>
+<vertex x="33.02" y="0"/>
+<vertex x="0" y="0"/>
+</polygon>
+<via x="21.2725" y="19.05" extent="1-16" drill="0.3302" diameter="0.1778"/>
+<via x="21.2725" y="17.145" extent="1-16" drill="0.3302" diameter="0.1778"/>
+<via x="20.32" y="17.145" extent="1-16" drill="0.3302" diameter="0.1778"/>
+<via x="19.3675" y="19.05" extent="1-16" drill="0.3302" diameter="0.1778"/>
+<via x="19.3675" y="10.4775" extent="1-16" drill="0.3302" diameter="0.1778"/>
+<via x="19.3675" y="8.5725" extent="1-16" drill="0.3302" diameter="0.1778"/>
+<via x="21.9075" y="11.7475" extent="1-16" drill="0.3302" diameter="0.1778"/>
+<via x="20.955" y="7.62" extent="1-16" drill="0.3302" diameter="0.1778"/>
+<via x="21.9075" y="7.62" extent="1-16" drill="0.3302" diameter="0.1778"/>
+<via x="4.1275" y="6.6675" extent="1-16" drill="0.3302" diameter="0.1778"/>
+<via x="5.08" y="8.5725" extent="1-16" drill="0.3302" diameter="0.1778"/>
+<via x="5.08" y="7.62" extent="1-16" drill="0.3302" diameter="0.1778"/>
+<via x="4.1275" y="7.62" extent="1-16" drill="0.3302" diameter="0.1778"/>
+<via x="26.035" y="19.685" extent="1-16" drill="0.3302" diameter="0.1778"/>
+<via x="26.9875" y="19.685" extent="1-16" drill="0.3302" diameter="0.1778"/>
+<via x="24.13" y="19.685" extent="1-16" drill="0.3302" diameter="0.1778"/>
+<via x="23.1775" y="19.685" extent="1-16" drill="0.3302" diameter="0.1778"/>
+<via x="22.225" y="19.685" extent="1-16" drill="0.3302" diameter="0.1778"/>
+<via x="19.3675" y="18.0975" extent="1-16" drill="0.3302" diameter="0.1778"/>
+<via x="20.32" y="18.0975" extent="1-16" drill="0.3302" diameter="0.1778"/>
+<via x="25.0825" y="19.685" extent="1-16" drill="0.3302" diameter="0.1778"/>
+<via x="20.32" y="19.05" extent="1-16" drill="0.3302" diameter="0.1778"/>
+<via x="19.3675" y="9.525" extent="1-16" drill="0.3302" diameter="0.1778"/>
+<via x="4.1275" y="8.5725" extent="1-16" drill="0.3302" diameter="0.1778"/>
+<via x="6.0325" y="8.5725" extent="1-16" drill="0.3302" diameter="0.1778"/>
+<via x="6.0325" y="7.62" extent="1-16" drill="0.3302" diameter="0.1778"/>
+<via x="5.08" y="6.6675" extent="1-16" drill="0.3302" diameter="0.1778"/>
+<via x="6.0325" y="6.6675" extent="1-16" drill="0.3302" diameter="0.1778"/>
 </signal>
 <signal name="SW">
@@
 <contactref element="RFBT" pad="1"/>
 <contactref element="COUT" pad="2"/>
-<polygon width="0.27" layer="1" thermals="no">
-<vertex x="20.39" y="14.54"/>
-<vertex x="20.38" y="14.54"/>
-<vertex x="20.38" y="12.53"/>
+<polygon width="0.27" layer="1" thermals="no" rank="2">
+<vertex x="21.015" y="14.54"/>
+<vertex x="20.955" y="12.53"/>
 <vertex x="22.27" y="12.53"/>
 <vertex x="23.03" y="11.77"/>
 <vertex x="23.03" y="1.925"/>
 <vertex x="29.865" y="1.925"/>
-<vertex x="30.48" y="2.54"/>
-<vertex x="30.48" y="5.08"/>
+<vertex x="31.4325" y="3.4925"/>
+<vertex x="31.4325" y="5.08"/>
 <vertex x="28.89" y="6.67"/>
 <vertex x="28.89" y="10.84"/>
 <vertex x="26.15" y="14.55"/>
-<vertex x="20.38" y="14.55"/>
 </polygon>
 <contactref element="J4" pad="5"/>
@@
 <contactref element="+6" pad="2"/>
 <contactref element="R1" pad="1"/>
-<wire x1="30.48" y1="6.5532" x2="30.48" y2="9.9314" width="0.27" layer="1"/>
+<wire x1="30.48" y1="7.1882" x2="30.48" y2="9.9314" width="0.27" layer="1"/>
 </signal>
 </signals>
