File: v3/hydrogen.sch (EAGLE design)
At the start: 19 parts, among them U1 TPS61088VQFN20

Commit message: Hydrogen board v1r0 off to OSH park.
Parts:
- added H: 1, 32bits:PERIODIC_SYMBOL
Connections:
- net GND: now also U1.PGND@25
Other:
- moved on the sheet: +6, CVCC, R1
Changed lines of the file:
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@@
 <part name="R1" library="Vishay_By_element14_Batch_1" deviceset="CRCW1206200RJNEA" device="" value="200 Ohms"/>
 <part name="GND2" library="SparkFun-PowerSymbols" deviceset="GND" device=""/>
+<part name="H" library="32bits" deviceset="PERIODIC_SYMBOL" device="" value="1">
+<attribute name="DESC" value="rev.0"/>
+</part>
 </parts>
 <sheets>
@@
 <attribute name="NAME" x="142.0114" y="1.6256" size="2.0828" layer="95" ratio="10" rot="SR90"/>
 </instance>
-<instance part="CVCC" gate="A" x="50.8" y="15.24" smashed="yes" rot="R180">
-<attribute name="VALUE" x="51.8922" y="20.5232" size="2.1209" layer="96" ratio="10" rot="SR180"/>
-<attribute name="NAME" x="51.7144" y="12.4714" size="2.0828" layer="95" ratio="10" rot="SR180"/>
+<instance part="CVCC" gate="A" x="50.8" y="17.78" smashed="yes" rot="R180">
+<attribute name="VALUE" x="51.8922" y="23.0632" size="2.1209" layer="96" ratio="10" rot="SR180"/>
+<attribute name="NAME" x="51.7144" y="15.0114" size="2.0828" layer="95" ratio="10" rot="SR180"/>
 </instance>
 <instance part="RCOMP" gate="A" x="198.12" y="0" smashed="yes" rot="R90">
@@
 <instance part="J1" gate="G$1" x="160.02" y="60.96" rot="R180"/>
 <instance part="J4" gate="G$1" x="137.16" y="60.96" rot="R180"/>
-<instance part="+6" gate="A" x="187.96" y="78.74" smashed="yes" rot="R270">
-<attribute name="VALUE" x="184.7342" y="78.6892" size="1.778" layer="96" ratio="10" rot="SR180"/>
-<attribute name="NAME" x="191.262" y="82.1436" size="2.0828" layer="95" ratio="10" rot="SR270"/>
-</instance>
-<instance part="R1" gate="A" x="187.96" y="96.52" smashed="yes" rot="R270">
-<attribute name="VALUE" x="182.7784" y="98.3742" size="1.778" layer="96" ratio="10" rot="SR270"/>
-<attribute name="NAME" x="190.7286" y="95.5294" size="2.0828" layer="95" ratio="10" rot="SR270"/>
-</instance>
-<instance part="GND2" gate="1" x="187.96" y="55.88"/>
+<instance part="+6" gate="A" x="195.58" y="58.42" smashed="yes" rot="R270">
+<attribute name="VALUE" x="192.3542" y="58.3692" size="1.778" layer="96" ratio="10" rot="SR180"/>
+<attribute name="NAME" x="198.882" y="61.8236" size="2.0828" layer="95" ratio="10" rot="SR270"/>
+</instance>
+<instance part="R1" gate="A" x="195.58" y="76.2" smashed="yes" rot="R270">
+<attribute name="VALUE" x="190.3984" y="78.0542" size="1.778" layer="96" ratio="10" rot="SR270"/>
+<attribute name="NAME" x="198.3486" y="75.2094" size="2.0828" layer="95" ratio="10" rot="SR270"/>
+</instance>
+<instance part="GND2" gate="1" x="195.58" y="43.18"/>
+<instance part="H" gate="G$1" x="121.92" y="83.82">
+<attribute name="DESC" x="121.92" y="83.82" size="1.778" layer="96" display="off"/>
+</instance>
 </instances>
 <busses>
@@
 <pinref part="GND1" gate="1" pin="GND"/>
 <wire x1="114.3" y1="-27.94" x2="58.42" y2="-27.94" width="0.1524" layer="91"/>
-<wire x1="58.42" y1="-27.94" x2="58.42" y2="10.16" width="0.1524" layer="91"/>
+<wire x1="58.42" y1="-27.94" x2="58.42" y2="12.7" width="0.1524" layer="91"/>
 <pinref part="U1" gate="G$1" pin="PGND@21"/>
-<wire x1="58.42" y1="10.16" x2="88.9" y2="10.16" width="0.1524" layer="91"/>
+<wire x1="58.42" y1="12.7" x2="88.9" y2="12.7" width="0.1524" layer="91"/>
 <junction x="58.42" y="-27.94"/>
 <pinref part="CIN" gate="A" pin="C1"/>
@@
 <junction x="33.02" y="-27.94"/>
 <pinref part="CVCC" gate="A" pin="C2"/>
-<wire x1="43.18" y1="15.24" x2="40.64" y2="15.24" width="0.1524" layer="91"/>
-<wire x1="40.64" y1="15.24" x2="40.64" y2="-27.94" width="0.1524" layer="91"/>
+<wire x1="43.18" y1="17.78" x2="40.64" y2="17.78" width="0.1524" layer="91"/>
+<wire x1="40.64" y1="17.78" x2="40.64" y2="-27.94" width="0.1524" layer="91"/>
 <junction x="40.64" y="-27.94"/>
 <pinref part="U1" gate="G$1" pin="NC@11"/>
@@
 <junction x="220.98" y="-27.94"/>
 <pinref part="U1" gate="G$1" pin="PGND@22"/>
+<wire x1="88.9" y1="12.7" x2="88.9" y2="10.16" width="0.1524" layer="91"/>
+<junction x="88.9" y="12.7"/>
+<pinref part="U1" gate="G$1" pin="PGND@23"/>
 <wire x1="88.9" y1="10.16" x2="88.9" y2="7.62" width="0.1524" layer="91"/>
 <junction x="88.9" y="10.16"/>
-<pinref part="U1" gate="G$1" pin="PGND@23"/>
+<pinref part="U1" gate="G$1" pin="PGND@24"/>
 <wire x1="88.9" y1="7.62" x2="88.9" y2="5.08" width="0.1524" layer="91"/>
 <junction x="88.9" y="7.62"/>
-<pinref part="U1" gate="G$1" pin="PGND@24"/>
-<wire x1="88.9" y1="5.08" x2="88.9" y2="2.54" width="0.1524" layer="91"/>
-<junction x="88.9" y="5.08"/>
 <pinref part="U1" gate="G$1" pin="AGND"/>
 <wire x1="124.46" y1="5.08" x2="124.46" y2="-27.94" width="0.1524" layer="91"/>
 <junction x="124.46" y="-27.94"/>
+<pinref part="U1" gate="G$1" pin="PGND@25"/>
+<wire x1="88.9" y1="5.08" x2="88.9" y2="2.54" width="0.1524" layer="91"/>
+<junction x="88.9" y="5.08"/>
 </segment>
 <segment>
@@
 <pinref part="+6" gate="A" pin="1"/>
 <pinref part="GND2" gate="1" pin="GND"/>
-<wire x1="187.96" y1="68.58" x2="187.96" y2="58.42" width="0.1524" layer="91"/>
+<wire x1="195.58" y1="48.26" x2="195.58" y2="45.72" width="0.1524" layer="91"/>
 </segment>
 </net>
@@
 <pinref part="U1" gate="G$1" pin="SW@7"/>
 <pinref part="U1" gate="G$1" pin="SW@6"/>
-<wire x1="88.9" y1="25.4" x2="88.9" y2="27.94" width="0.1524" layer="91"/>
+<wire x1="88.9" y1="27.94" x2="88.9" y2="30.48" width="0.1524" layer="91"/>
 <pinref part="U1" gate="G$1" pin="SW@5"/>
-<wire x1="88.9" y1="27.94" x2="88.9" y2="30.48" width="0.1524" layer="91"/>
-<junction x="88.9" y="27.94"/>
-<pinref part="U1" gate="G$1" pin="SW@4"/>
 <wire x1="88.9" y1="30.48" x2="88.9" y2="33.02" width="0.1524" layer="91"/>
 <junction x="88.9" y="30.48"/>
+<pinref part="U1" gate="G$1" pin="SW@4"/>
+<wire x1="88.9" y1="33.02" x2="88.9" y2="35.56" width="0.1524" layer="91"/>
 <junction x="88.9" y="33.02"/>
-<wire x1="88.9" y1="33.02" x2="88.9" y2="63.5" width="0.1524" layer="91"/>
+<junction x="88.9" y="35.56"/>
+<wire x1="88.9" y1="35.56" x2="88.9" y2="63.5" width="0.1524" layer="91"/>
 <pinref part="CBST" gate="A" pin="C2"/>
 <wire x1="104.14" y1="58.42" x2="104.14" y2="63.5" width="0.1524" layer="91"/>
@@
 <segment>
 <pinref part="U1" gate="G$1" pin="VIN"/>
-<wire x1="88.9" y1="17.78" x2="63.5" y2="17.78" width="0.1524" layer="91"/>
-<wire x1="63.5" y1="17.78" x2="63.5" y2="76.2" width="0.1524" layer="91"/>
+<wire x1="88.9" y1="20.32" x2="63.5" y2="20.32" width="0.1524" layer="91"/>
+<wire x1="63.5" y1="20.32" x2="63.5" y2="76.2" width="0.1524" layer="91"/>
 <pinref part="L1" gate="A" pin="2"/>
 <wire x1="63.5" y1="76.2" x2="71.12" y2="76.2" width="0.1524" layer="91"/>
@@
 <pinref part="U1" gate="G$1" pin="VCC"/>
 <pinref part="CVCC" gate="A" pin="C1"/>
-<wire x1="88.9" y1="15.24" x2="50.8" y2="15.24" width="0.1524" layer="91"/>
+<wire x1="88.9" y1="17.78" x2="50.8" y2="17.78" width="0.1524" layer="91"/>
 </segment>
 </net>
@@
 <segment>
 <pinref part="R1" gate="A" pin="2"/>
-<wire x1="187.96" y1="96.52" x2="187.96" y2="104.14" width="0.1524" layer="91"/>
-<label x="185.42" y="106.68" size="1.778" layer="95"/>
+<wire x1="195.58" y1="76.2" x2="195.58" y2="83.82" width="0.1524" layer="91"/>
+<label x="193.04" y="86.36" size="1.778" layer="95"/>
 </segment>
 </net>
@@
 <segment>
 <pinref part="RT" gate="A" pin="1"/>
-<wire x1="76.2" y1="45.72" x2="76.2" y2="20.32" width="0.1524" layer="91"/>
+<wire x1="76.2" y1="45.72" x2="76.2" y2="22.86" width="0.1524" layer="91"/>
 <pinref part="U1" gate="G$1" pin="FSW"/>
-<wire x1="76.2" y1="20.32" x2="88.9" y2="20.32" width="0.1524" layer="91"/>
+<wire x1="76.2" y1="22.86" x2="88.9" y2="22.86" width="0.1524" layer="91"/>
 </segment>
 </net>
@@
 <segment>
 <pinref part="U1" gate="G$1" pin="EN"/>
-<wire x1="88.9" y1="12.7" x2="78.74" y2="12.7" width="0.1524" layer="91"/>
-<label x="79.248" y="12.954" size="1.778" layer="95"/>
+<wire x1="88.9" y1="15.24" x2="78.74" y2="15.24" width="0.1524" layer="91"/>
+<label x="78.486" y="15.494" size="1.778" layer="95"/>
 </segment>
 <segment>
@@
 <pinref part="+6" gate="A" pin="2"/>
 <pinref part="R1" gate="A" pin="1"/>
-<wire x1="187.96" y1="78.74" x2="187.96" y2="83.82" width="0.1524" layer="91"/>
-</segment>
-</net>
+<wire x1="195.58" y1="58.42" x2="195.58" y2="63.5" width="0.1524" layer="91"/>
+</segment>
+</net>
