File: v3/lithium.sch (EAGLE design)
At the start: 31 parts, among them U1 TPS61088VQFN20, U2 TPS63051RMW, U3 SI2301BDS-T1-E3, U4 TPS2113APWR

Commit message: Significant completion of scheamtic.
Parts:
- removed U$2: MCP73833-FCI/UN, 32bits:MCP73833-FCI/UN
- added BATT, USB: 597-3311-407F, Dialight_By_element14_Batch_1:597-3311-407F
- added C1, C2: 1.0uF, SparkFun-Capacitors:1.0UF-0402-16V-10%
- added C3, C4: 0.1uF, SparkFun-Capacitors:0.1UF-0402-16V-10%
- added CHG: 597-3111-407F, Dialight_By_element14_Batch_1:597-3111-407F
- added DONE: 597-3401-407F, Dialight_By_element14_Batch_1:597-3401-407F
- added J1: batt, SparkFun-Connectors:CONN_02-JST-2MM-SMT
- added R3: 10K Ohms, Vishay_By_element14_Batch_1:CRCW040210K0FKED
- added R4: 1K Ohm, Vishay_By_element14_Batch_1:CRCW04021K00JNED
- added R5, R6, R7: 100 Ohms, Yageo_By_element14_Batch_1:9C04021A1000FLHF3
- added R8: 22, SparkFun-Resistors:22OHM-0402-1/10W-1%
- added R9: 200 Ohms, Vishay_By_element14_Batch_1:CRCW1206200RJNEA
- added RPG1: 100K Ohms, Vishay_By_element14_Batch_1:CRCW0603100KFKEA
- added S1: AS11CH, 32bits:AS11CH
- added U5: MCP73833-FCI/UN, 32bits:MCP73833-FCI/UN
- J3: value (none) -> robo
Connections:
- removed net VIN: CIN.C2, CIN1.C2, CIN2.C2, L1.2, U1.VIN, U2.ILIM0, U2.VIN
- new net N$10: BATT.2, R9.1
- new net N$11: S1.P$1, U4.OUT
- new net N$2: R8.2, U4.ILIM
- new net N$5: R4.1, U5.PROG
- new net N$6: R3.1, U5.THERM
- new net N$7: CHG.2, R5.R1
- new net N$8: DONE.2, R6.R1
- new net N$9: R7.R1, USB.2
- new net STAT: BATT.1, RPG1.2, U4.STAT
- new net STAT1: CHG.1, U5.STAT1
- new net STAT2: DONE.1, U5.STAT2
- new net U5_NPG: U5.!PG, USB.1
- new net VBAT: C2.1, C4.1, J1.1, U4.IN1, U5.VBAT, U5.VBAT_2
- new net VCC: CIN.C2, CIN1.C2, CIN2.C2, L1.2, R9.2, RPG1.1, S1.P$2, U1.VIN, U2.ILIM0, U2.VIN
- new net VUSB: C1.1, C3.1, R5.R2, R6.R2, R7.R2, U4.IN2, U5.VDD, U5.VDD_2
- net GND: now also C1.2, C2.2, C3.2, C4.2, J1.2, R3.2, R4.2, R8.1, U4.!EN, U4.GND, U4.VSNS, U5.VSS
Other:
- moved on the sheet: +3.3, +6, R1, R2, U3, U4

Commit message: Lego module mechanical and 5v rail
Switching to a 5v supply from the 3.3. Will use an LDO on the motor board to get 3.3. from the 5.
In-general, committing to a BB green/ROS controller for this robot.
Parts:
- removed CIN1, COUT1, COUTX: 10uF, Murata_By_element14_Batch_1:GRM188R60J106ME47D
- removed CSS: 1.3nF, Kemet_By_element14_Batch_1:C0402C132J5GACTU
- removed J3: robo, SparkFun-Connectors:CONN_10X2
- removed RPG: 100K Ohms, Vishay_By_element14_Batch_1:CRCW0603100KFKEA
- removed U2: TPS63051RMW, 32bits:TPS6305X
- added C5: 10 nF, Kemet_By_element14_Batch_1:C0402C103K5RACTU
- added C6: 0.22µF, AVX_By_element14_Batch_1:0306ZC224MAT2A
- added P8-1-2: bb-extra-gnd, SparkFun-Connectors:CONN_02
- added P8-27-46: robo, SparkFun-Connectors:CONN_10X2
- added P9-1-10: bb-pwr, SparkFun-Connectors:CONN_05X2PTH
- added P9-39-46: bb-extra-gnd, SparkFun-Connectors:CONN_04X2
- added U6: TPS61230A, 32bits:TPS61230A
- L2: value AISC-1008-1R5J-T -> 1.0 uH; device 32bits:AISC-1008-1R5J-T -> Bourns_By_element14_Batch_1:PM1210-1R0J-RC
- S1: value AS11CH -> PWR
Connections:
- net LED_ANODE renamed LA_6
- net N$10 renamed LA_BATT
- net N$4 renamed LA_3_3
- net N$7 renamed LA_CHG
- net N$8 renamed LA_DONE
- net N$9 renamed LA_USB
- removed net L1: L2.2, U2.L1
- removed net L2: L2.1, U2.L2
- removed net SS1: CSS.C2, U2.SS
- new net N$4: C5.C1, U6.CBST
- new net N$7: C5.C2, L2.1, U6.SW
- new net N$8: L2.2, U6.EN, U6.VIN
- net +3.3: now also P8-27-46.3, P8-27-46.4, P9-1-10.3, P9-1-10.4; no longer COUT1.C2, COUTX.C2, RPG.1, U2.FB, U2.VOUT
- net +6: now also P8-27-46.5, P8-27-46.6
- net EN: no longer U2.EN
- net GND: now also P8-1-2.1, P8-1-2.2, P8-27-46.1, P8-27-46.2, P9-1-10.1, P9-1-10.2, P9-39-46.5, P9-39-46.6, P9-39-46.7, P9-39-46.8; no longer CIN1.C1, COUT1.C1, COUTX.C1, CSS.C1, U2.GND@2, U2.GND@9, U2.MODE
- net NPG: no longer RPG.2, U2.PG
- net VCC: no longer CIN1.C2, U2.ILIM0, U2.VIN

Commit message: Progress on Lithium board.
Parts:
- removed C6: 0.22µF, AVX_By_element14_Batch_1:0306ZC224MAT2A
- removed J1: batt, SparkFun-Connectors:CONN_02-JST-2MM-SMT
- removed R7: 100 Ohms, Yageo_By_element14_Batch_1:9C04021A1000FLHF3
- removed R9: 200 Ohms, Vishay_By_element14_Batch_1:CRCW1206200RJNEA
- removed U3: SI2301BDS-T1-E3, Vishay_By_element14_Batch_1:SI2301BDS-T1-E3
- added U5_R1: 1K Ohm, Vishay_By_element14_Batch_1:CRCW04021K00JNED
- added U5_R2: 10K Ohms, Vishay_By_element14_Batch_1:CRCW120610K0JNEA
- added U6_CFF: 10pF, Kemet_By_element14_Batch_1:C0603C100J5GACTU
- added U6_CIN: 22uF, Murata_By_element14_Batch_1:GRM21BR60J226ME39L
- added U6_COUT: 22uF, Murata_By_element14_Batch_1:GRM32ER61C226KE20L
- added U6_RFBB: 100K Ohms, Vishay_By_element14_Batch_1:CRCW0402100KFKED
- added U6_RFBT: 316K Ohms, Vishay_By_element14_Batch_1:CRCW0402316KFKED
- 5V, BATT, USB: value 597-3311-407F -> QTLP650C-4
- CHG: value 597-3111-407F -> QTLP650C-7
- DONE: value 597-3401-407F -> QTLP650C-3
- MOTORS: value 597-3311-402F -> QTLP650C-B
- P8-27-46: value robo -> motors
- R1: value 200 Ohms -> 15 Ohm; device Vishay_By_element14_Batch_1:CRCW1206200RJNEA -> Vishay_By_element14_Batch_1:CRCW080515R0JNEA
- R2, R5, R6: value 100 Ohms -> 15 Ohm; device Yageo_By_element14_Batch_1:9C04021A1000FLHF3 -> Vishay_By_element14_Batch_1:CRCW080515R0JNEA
- R3: value 10K Ohms -> 15 Ohm; device Vishay_By_element14_Batch_1:CRCW040210K0FKED -> Vishay_By_element14_Batch_1:CRCW080515R0JNEA
- R4: value 1K Ohm -> 15 Ohm; device Vishay_By_element14_Batch_1:CRCW04021K00JNED -> Vishay_By_element14_Batch_1:CRCW080515R0JNEA
- U1: device digikey:TPS61088VQFN20 -> 32bits:TPS61088VQFN20
- renumbered +3.3 to 5V, +6 to MOTORS, C1 to U5_C1, C2 to U5_C2, C22 to U1_C22, C3 to U4_C3, C4 to U4_C4, C5 to U6_CBST, CBST to U1_CBST, CCOMP to U1_CCOMP, CCOMP2 to U1_CCOMP2, CIN to U1_CIN, CIN2 to U1_CIN2, COUT to U1_COUT, CVCC to U1_CVCC, L1 to U1_L1, R8 to U4_R8, RCOMP to U1_RCOMP, RFBB to U1_RFBB, RFBT to U1_RFBT, RLIM to U1_RLIM, RPG1 to U4_RPG, RT to U1_RT
Connections:
- net COMP renamed U1_COMP
- net N$11 renamed S1_U4OUT
- net N$2 renamed U4_ILIM
- net STAT renamed U4_STAT
- removed net +3.3: P8-27-46.3, P8-27-46.4, P9-1-10.3, P9-1-10.4, R2.R2
- removed net +6: P8-27-46.5, P8-27-46.6, R1.2, U1.VOUT@14, U1.VOUT@15, U1.VOUT@16, U1_COUT.C2, U1_RFBT.R1
- removed net EN: U1.EN
- removed net LA_3_3: 5V.2, R2.R1
- removed net MODE: U1.MODE
- removed net N$3: 5V.1, U3.D
- removed net N$5: R4.1, U5.PROG
- removed net N$6: R3.1, U5.THERM
- removed net N$8: L2.2, U6.EN, U6.VIN
- removed net NPG: U3.G
- removed net VCC1: U1.VCC, U1_CVCC.C1
- new net LA_5: 5V.2, R1.1
- new net MOT_6V: P8-27-46.17, P8-27-46.18, R2.2, U1.VOUT@14, U1.VOUT@15, U1.VOUT@16, U1_COUT.C2, U1_RFBT.R1
- new net N$9: U6.FB, U6_CFF.C1, U6_RFBB.1, U6_RFBT.2
- new net SYS_5V: P9-1-10.7, P9-1-10.8, R1.2, U6.VOUT, U6_CFF.C2, U6_COUT.C2, U6_RFBT.1
- new net U1_VCC: U1.EN, U1.VCC, U1_CVCC.C1
- new net U5_PROG: U5.PROG, U5_R1.1
- new net U5_THERM: P8-27-46.5, U5.THERM, U5_R2.1
- net GND: now also 5V.1, P8-27-46.15, P8-27-46.16, P8-27-46.19, P8-27-46.20, U5_R1.2, U5_R2.2, U6.GND, U6_CIN.C1, U6_COUT.C1, U6_RFBB.2; no longer J1.2, R3.2, R4.2, U3.S
- net LA_6: now also R2.1; no longer R1.1
- net LA_BATT: now also R6.1; no longer R9.1
- net LA_CHG: now also R3.1; no longer R5.R1
- net LA_DONE: now also R4.1; no longer R6.R1
- net LA_USB: now also R5.1; no longer R7.R1
- net VBAT: now also P8-27-46.3, P8-27-46.4; no longer J1.1
- net VCC: now also L2.2, R6.2, U6.EN, U6.VIN, U6_CIN.C2; no longer R9.2
- net VUSB: now also P8-27-46.13, P8-27-46.14, R3.2, R4.2, R5.2; no longer R5.R2, R6.R2, R7.R2
Other:
- moved on the sheet: R1, R2, R3, R4, R5, R6, S1

Commit message: Significant completion of Lithium layout.
TODO:
1. reverse voltage protection.
2. silk screen
Parts:
- removed U4_R8: 22, SparkFun-Resistors:22OHM-0402-1/10W-1%
- removed U5_R2: 10K Ohms, Vishay_By_element14_Batch_1:CRCW120610K0JNEA
- added J1: batt, SparkFun-Connectors:CONN_02-JST-2MM-SMT
- added R7: 22 Ohms, Vishay_By_element14_Batch_1:CRCW040222R0JNED
- added R8: 0Ohm, Vishay_By_element14_Batch_1:CRCW08050000Z0EB
- added R9: 10k, 32bits:NTHS1206N02N1002JE
Connections:
- net N$4 renamed U6_CBST
- net N$7 renamed U6_SW
- net N$9 renamed U6_FB
- removed net GND: 5V.1, MOTORS.1, P8-1-2.1, P8-1-2.2, P8-27-46.1, P8-27-46.15, P8-27-46.16, P8-27-46.19, P8-27-46.2, P8-27-46.20, P9-1-10.1, P9-1-10.2, P9-39-46.5, P9-39-46.6, P9-39-46.7, P9-39-46.8, U1.AGND, U1.NC@11, U1.NC@12, U1.PGND@21, U1.PGND@22, U1.PGND@23, U1.PGND@24, U1.PGND@25, U1_C22.C1, U1_CCOMP.C1, U1_CCOMP2.C1, U1_CIN.C1, U1_CIN2.C1, U1_COUT.C1, U1_CVCC.C2, U1_RFBB.1, U1_RLIM.2, U4.!EN, U4.GND, U4.VSNS, U4_C3.2, U4_C4.2, U4_R8.1, U5.VSS, U5_C1.2, U5_C2.2, U5_R1.2, U5_R2.2, U6.GND, U6_CIN.C1, U6_COUT.C1, U6_RFBB.2
- new net COPU: 5V.1, J1.2, MOTORS.1, P8-1-2.1, P8-1-2.2, P8-27-46.1, P8-27-46.15, P8-27-46.16, P8-27-46.19, P8-27-46.2, P8-27-46.20, P9-1-10.1, P9-1-10.2, P9-39-46.5, P9-39-46.6, P9-39-46.7, P9-39-46.8, R7.2, R9.1, U1.AGND, U1.NC@11, U1.NC@12, U1.PGND@21, U1.PGND@22, U1.PGND@23, U1.PGND@24, U1.PGND@25, U1_C22.C1, U1_CCOMP.C1, U1_CCOMP2.C1, U1_CIN.C1, U1_CIN2.C1, U1_COUT.C1, U1_CVCC.C2, U1_RFBB.1, U1_RLIM.2, U4.!EN, U4.GND, U4.VSNS, U4_C3.2, U4_C4.2, U5.VSS, U5_C1.2, U5_C2.2, U5_R1.2, U6.GND, U6_CIN.C1, U6_COUT.C1, U6_RFBB.2
- new net LOCAL_VBAT: J1.1, R8.2
- net S1_U4OUT: now also S1.P$2; no longer S1.P$1
- net U4_ILIM: now also R7.1; no longer U4_R8.2
- net U5_THERM: now also P9-39-46.1, R9.2; no longer P8-27-46.5, U5_R2.1
- net VBAT: now also P9-39-46.3, P9-39-46.4, R8.1; no longer P8-27-46.3, P8-27-46.4
- net VCC: now also S1.P$1; no longer S1.P$2
Changed lines of the file:
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@@
 <?xml version="1.0" encoding="utf-8"?>
 <!DOCTYPE eagle SYSTEM "eagle.dtd">
-<eagle version="7.7.0">
+<eagle version="8.1.0">
 <drawing>
 <settings>
@@
 <part name="U4_C3" library="SparkFun-Capacitors" deviceset="0.1UF" device="-0402-16V-10%" value="0.1uF"/>
 <part name="U4_C4" library="SparkFun-Capacitors" deviceset="0.1UF" device="-0402-16V-10%" value="0.1uF"/>
-<part name="U4_R8" library="SparkFun-Resistors" deviceset="22OHM" device="-0402-1/10W-1%" value="22"/>
 <part name="BATT" library="Dialight_By_element14_Batch_1" deviceset="597-3311-407F" device="" value="QTLP650C-4"/>
 <part name="U4_RPG" library="Vishay_By_element14_Batch_1" deviceset="CRCW0603100KFKEA" device="" value="100K Ohms"/>
@@
 <part name="R5" library="Vishay_By_element14_Batch_1" deviceset="CRCW080515R0JNEA" device="" value="15 Ohm"/>
 <part name="R6" library="Vishay_By_element14_Batch_1" deviceset="CRCW080515R0JNEA" device="" value="15 Ohm"/>
-<part name="U5_R2" library="Vishay_By_element14_Batch_1" deviceset="CRCW120610K0JNEA" device="" value="10K Ohms"/>
+<part name="R7" library="Vishay_By_element14_Batch_1" deviceset="CRCW040222R0JNED" device="" value="22 Ohms"/>
+<part name="J1" library="SparkFun-Connectors" deviceset="CONN_02" device="-JST-2MM-SMT" value="batt"/>
+<part name="R8" library="Vishay_By_element14_Batch_1" deviceset="CRCW08050000Z0EB" device="" value="0Ohm"/>
+<part name="R9" library="32bits" deviceset="NTHS1206N02N1002JE" device="" value="10k"/>
 </parts>
 <sheets>
@@
 <instance part="U4_C3" gate="G$1" x="358.14" y="33.02"/>
 <instance part="U4_C4" gate="G$1" x="378.46" y="33.02"/>
-<instance part="U4_R8" gate="G$1" x="294.64" y="27.94" rot="R90"/>
 <instance part="BATT" gate="A" x="261.62" y="101.6" smashed="yes" rot="R270">
 <attribute name="VALUE" x="267.7668" y="104.9782" size="1.27" layer="96" ratio="10" rot="SR270"/>
@@
 <attribute name="NAME" x="264.3886" y="118.3894" size="2.0828" layer="95" ratio="10" rot="SR270"/>
 </instance>
-<instance part="U5_R2" gate="A" x="355.6" y="152.4" smashed="yes" rot="R90">
-<attribute name="VALUE" x="360.2736" y="152.3238" size="1.778" layer="96" ratio="10" rot="SR90"/>
-<attribute name="NAME" x="352.8314" y="153.3906" size="2.0828" layer="95" ratio="10" rot="SR90"/>
-</instance>
+<instance part="R7" gate="A" x="297.18" y="20.32" smashed="yes" rot="R90">
+<attribute name="VALUE" x="304.3936" y="22.2758" size="1.27" layer="96" ratio="10" rot="SR90"/>
+<attribute name="NAME" x="302.2854" y="22.3266" size="2.0828" layer="95" ratio="10" rot="SR90"/>
+</instance>
+<instance part="J1" gate="G$1" x="7.62" y="142.24"/>
+<instance part="R8" gate="A" x="25.4" y="142.24"/>
+<instance part="R9" gate="G$1" x="355.6" y="152.4" rot="R90"/>
 </instances>
 <busses>
 </busses>
 <nets>
-<net name="GND" class="0">
+<net name="COPU" class="0">
 <segment>
 <pinref part="GND1" gate="1" pin="GND"/>
@@
 <pinref part="U5_C2" gate="G$1" pin="2"/>
 <wire x1="368.3" y1="162.56" x2="368.3" y2="139.7" width="0.1524" layer="91"/>
+<pinref part="U5_C1" gate="G$1" pin="2"/>
 <wire x1="368.3" y1="139.7" x2="355.6" y2="139.7" width="0.1524" layer="91"/>
-<pinref part="U5_C1" gate="G$1" pin="2"/>
 <wire x1="355.6" y1="139.7" x2="337.82" y2="139.7" width="0.1524" layer="91"/>
 <wire x1="337.82" y1="139.7" x2="304.8" y2="139.7" width="0.1524" layer="91"/>
@@
 <wire x1="337.82" y1="147.32" x2="337.82" y2="139.7" width="0.1524" layer="91"/>
 <junction x="337.82" y="139.7"/>
-<wire x1="355.6" y1="152.4" x2="355.6" y2="139.7" width="0.1524" layer="91"/>
+<junction x="304.8" y="139.7"/>
+<pinref part="R9" gate="G$1" pin="1"/>
+<wire x1="355.6" y1="147.32" x2="355.6" y2="139.7" width="0.1524" layer="91"/>
 <junction x="355.6" y="139.7"/>
-<junction x="304.8" y="139.7"/>
-<pinref part="U5_R2" gate="A" pin="2"/>
 </segment>
 <segment>
@@
 <junction x="322.58" y="15.24"/>
 <pinref part="U4_C4" gate="G$1" pin="2"/>
-<wire x1="287.02" y1="15.24" x2="294.64" y2="15.24" width="0.1524" layer="91"/>
-<wire x1="294.64" y1="15.24" x2="322.58" y2="15.24" width="0.1524" layer="91"/>
+<wire x1="287.02" y1="15.24" x2="297.18" y2="15.24" width="0.1524" layer="91"/>
+<wire x1="297.18" y1="15.24" x2="322.58" y2="15.24" width="0.1524" layer="91"/>
 <wire x1="350.52" y1="15.24" x2="358.14" y2="15.24" width="0.1524" layer="91"/>
 <wire x1="358.14" y1="15.24" x2="378.46" y2="15.24" width="0.1524" layer="91"/>
@@
 <wire x1="358.14" y1="30.48" x2="358.14" y2="15.24" width="0.1524" layer="91"/>
 <junction x="358.14" y="15.24"/>
-<pinref part="U4_R8" gate="G$1" pin="1"/>
-<wire x1="294.64" y1="22.86" x2="294.64" y2="15.24" width="0.1524" layer="91"/>
-<junction x="294.64" y="15.24"/>
 <pinref part="U4" gate="A" pin="VSNS"/>
 <wire x1="297.18" y1="40.64" x2="287.02" y2="40.64" width="0.1524" layer="91"/>
 <wire x1="287.02" y1="40.64" x2="287.02" y2="15.24" width="0.1524" layer="91"/>
 <junction x="287.02" y="15.24"/>
+<pinref part="R7" gate="A" pin="2"/>
+<wire x1="297.18" y1="20.32" x2="297.18" y2="15.24" width="0.1524" layer="91"/>
+<junction x="297.18" y="15.24"/>
 </segment>
 <segment>
@@
 <wire x1="0" y1="165.1" x2="-7.62" y2="165.1" width="0.1524" layer="91"/>
 <label x="-7.874" y="165.354" size="1.778" layer="95"/>
+</segment>
+<segment>
+<pinref part="J1" gate="G$1" pin="2"/>
+<wire x1="15.24" y1="144.78" x2="25.4" y2="144.78" width="0.1524" layer="91"/>
+<label x="20.32" y="145.288" size="1.778" layer="95"/>
 </segment>
 </net>
@@
 </segment>
 <segment>
-<wire x1="360.68" y1="50.8" x2="360.68" y2="81.28" width="0.1524" layer="91"/>
+<wire x1="360.68" y1="68.58" x2="360.68" y2="81.28" width="0.1524" layer="91"/>
 <label x="358.14" y="81.788" size="1.778" layer="95"/>
-<pinref part="S1" gate="G$1" pin="P$2"/>
+<pinref part="S1" gate="G$1" pin="P$1"/>
 </segment>
 <segment>
@@
 </segment>
 <segment>
-<pinref part="P8-27-46" gate="G$1" pin="4"/>
-<wire x1="15.24" y1="180.34" x2="22.86" y2="180.34" width="0.1524" layer="91"/>
-<label x="17.526" y="180.594" size="1.778" layer="95"/>
-</segment>
-<segment>
-<pinref part="P8-27-46" gate="G$1" pin="3"/>
-<wire x1="0" y1="180.34" x2="-7.62" y2="180.34" width="0.1524" layer="91"/>
-<label x="-9.398" y="180.594" size="1.778" layer="95"/>
+<pinref part="P9-39-46" gate="G$1" pin="3"/>
+<wire x1="-38.1" y1="165.1" x2="-48.26" y2="165.1" width="0.1524" layer="91"/>
+<label x="-48.006" y="165.354" size="1.778" layer="95"/>
+</segment>
+<segment>
+<pinref part="P9-39-46" gate="G$1" pin="4"/>
+<wire x1="-22.86" y1="165.1" x2="-12.7" y2="165.1" width="0.1524" layer="91"/>
+<label x="-18.796" y="165.608" size="1.778" layer="95"/>
+</segment>
+<segment>
+<pinref part="R8" gate="A" pin="1"/>
+<wire x1="38.1" y1="142.24" x2="48.26" y2="142.24" width="0.1524" layer="91"/>
+<label x="42.164" y="142.748" size="1.778" layer="95"/>
 </segment>
 </net>
@@
 <segment>
 <pinref part="U5" gate="A" pin="!PG"/>
-<wire x1="335.28" y1="162.56" x2="345.44" y2="162.56" width="0.1524" layer="91"/>
 <label x="340.36" y="160.274" size="1.778" layer="95"/>
+<wire x1="347.98" y1="162.56" x2="335.28" y2="162.56" width="0.1524" layer="91"/>
 </segment>
 <segment>
@@
 <wire x1="246.38" y1="101.6" x2="246.38" y2="106.68" width="0.1524" layer="91"/>
 <pinref part="R5" gate="A" pin="1"/>
-</segment>
-</net>
-<net name="U4_ILIM" class="0">
-<segment>
-<pinref part="U4" gate="A" pin="ILIM"/>
-<pinref part="U4_R8" gate="G$1" pin="2"/>
-<wire x1="297.18" y1="38.1" x2="294.64" y2="38.1" width="0.1524" layer="91"/>
-<wire x1="294.64" y1="38.1" x2="294.64" y2="33.02" width="0.1524" layer="91"/>
 </segment>
 </net>
@@
 <pinref part="U4" gate="A" pin="OUT"/>
 <wire x1="347.98" y1="43.18" x2="360.68" y2="43.18" width="0.1524" layer="91"/>
-<wire x1="360.68" y1="43.18" x2="360.68" y2="68.58" width="0.1524" layer="91"/>
-<pinref part="S1" gate="G$1" pin="P$1"/>
-<junction x="360.68" y="68.58"/>
-</segment>
-</net>
-<net name="N$4" class="0">
+<wire x1="360.68" y1="43.18" x2="360.68" y2="50.8" width="0.1524" layer="91"/>
+<pinref part="S1" gate="G$1" pin="P$2"/>
+<junction x="360.68" y="50.8"/>
+</segment>
+</net>
+<net name="U6_CBST" class="0">
 <segment>
 <pinref part="U6" gate="G$1" pin="CBST"/>
@@
 </segment>
 </net>
-<net name="N$7" class="0">
+<net name="U6_SW" class="0">
 <segment>
 <pinref part="U6_CBST" gate="A" pin="C2"/>
@@
 </segment>
 </net>
-<net name="N$9" class="0">
+<net name="U6_FB" class="0">
 <segment>
 <pinref part="U6" gate="G$1" pin="FB"/>
@@
 <wire x1="335.28" y1="165.1" x2="355.6" y2="165.1" width="0.1524" layer="91"/>
 <label x="342.646" y="165.862" size="1.778" layer="95"/>
-<pinref part="U5_R2" gate="A" pin="1"/>
-</segment>
-<segment>
-<pinref part="P8-27-46" gate="G$1" pin="5"/>
-<wire x1="0" y1="177.8" x2="-7.62" y2="177.8" width="0.1524" layer="91"/>
-<label x="-12.954" y="178.054" size="1.778" layer="95"/>
-</segment>
-</net>
+<pinref part="R9" gate="G$1" pin="2"/>
+<wire x1="355.6" y1="165.1" x2="355.6" y2="157.48" width="0.1524" layer="91"/>
+</segment>
+<segment>
+<pinref part="P9-39-46" gate="G$1" pin="1"/>
+<wire x1="-38.1" y1="167.64" x2="-48.26" y2="167.64" width="0.1524" layer="91"/>
+<label x="-53.594" y="167.894" size="1.778" layer="95"/>
+</segment>
+</net>
+<net name="U4_ILIM" class="0">
+<segment>
+<pinref part="U4" gate="A" pin="ILIM"/>
+<pinref part="R7" gate="A" pin="1"/>
+<wire x1="297.18" y1="38.1" x2="297.18" y2="33.02" width="0.1524" layer="91"/>
+</segment>
+</net>
+<net name="LOCAL_VBAT" class="0">
+<segment>
+<pinref part="J1" gate="G$1" pin="1"/>
+<pinref part="R8" gate="A" pin="2"/>
+<wire x1="15.24" y1="142.24" x2="25.4" y2="142.24" width="0.1524" layer="91"/>
+</segment>
+</net>
