File: v3/lithium.sch (EAGLE design)
At the start: 53 parts, among them J1 batt, P8-1-2 bb-extra-gnd, P8-27-46 motors, P9-1-10 bb-pwr, P9-39-46 bb-extra-gnd, U1 TPS61088VQFN20, U1_C22 8.2nF, U1_CBST 100nF, U1_CCOMP 680PF, U1_CCOMP2 36pF, U1_CIN 0.47uF, U1_CIN2 100nF, U1_COUT 0.47uF, U1_CVCC 1uF, U1_L1 DR73-1R0-R, U1_RCOMP 38.3K Ohms, U1_RFBB 118K Ohms, U1_RFBT 470K Ohms, U1_RLIM 102K Ohms, U1_RT 261K Ohms, U4 TPS2113APWR, U4_C3 0.1uF, U4_C4 0.1uF, U4_RPG 100K Ohms, U5 MCP73833-FCI/UN, U5_C1 1.0uF, U5_C2 1.0uF, U5_R1 1K Ohm, U6 TPS61230A, U6_CBST 10 nF, U6_CFF 10pF, U6_CIN 22uF, U6_COUT 22uF, U6_RFBB 100K Ohms, U6_RFBT 316K Ohms

Commit message: Moving away from bb ideas.
Parts:
- removed P8-1-2: bb-extra-gnd, SparkFun-Connectors:CONN_02
- removed P9-39-46: bb-extra-gnd, SparkFun-Connectors:CONN_04X2
- added J2: 2X4-0.01"(2.54MM)-HEADERS, 32bits:2X4-0.01"(2.54MM)-HEADERS
- added U2: SI2312BDS-T1-GE3, 32bits:SI2312BDS-T1-GE3
Connections:
- removed net COPU: 5V.1, J1.2, MOTORS.1, P8-1-2.1, P8-1-2.2, P8-27-46.1, P8-27-46.15, P8-27-46.16, P8-27-46.19, P8-27-46.2, P8-27-46.20, P9-1-10.1, P9-1-10.2, P9-39-46.5, P9-39-46.6, P9-39-46.7, P9-39-46.8, R7.2, R9.1, U1.AGND, U1.NC@11, U1.NC@12, U1.PGND@21, U1.PGND@22, U1.PGND@23, U1.PGND@24, U1.PGND@25, U1_C22.C1, U1_CCOMP.C1, U1_CCOMP2.C1, U1_CIN.C1, U1_CIN2.C1, U1_COUT.C1, U1_CVCC.C2, U1_RFBB.1, U1_RLIM.2, U4.!EN, U4.GND, U4.VSNS, U4_C3.2, U4_C4.2, U5.VSS, U5_C1.2, U5_C2.2, U5_R1.2, U6.GND, U6_CIN.C1, U6_COUT.C1, U6_RFBB.2
- new net GND: 5V.1, J1.2, J2.5, J2.6, J2.7, MOTORS.1, P8-27-46.1, P8-27-46.15, P8-27-46.16, P8-27-46.19, P8-27-46.2, P8-27-46.20, P9-1-10.1, P9-1-10.2, R7.2, R9.1, U1.AGND, U1.NC@11, U1.NC@12, U1.PGND@21, U1.PGND@22, U1.PGND@23, U1.PGND@24, U1.PGND@25, U1_C22.C1, U1_CCOMP.C1, U1_CCOMP2.C1, U1_CIN.C1, U1_CIN2.C1, U1_COUT.C1, U1_CVCC.C2, U1_RFBB.1, U1_RLIM.2, U4.!EN, U4.GND, U4.VSNS, U4_C3.2, U4_C4.2, U5.VSS, U5_C1.2, U5_C2.2, U5_R1.2, U6.GND, U6_CIN.C1, U6_COUT.C1, U6_RFBB.2
- new net N$4: J2.8
- net U5_THERM: now also J2.1; no longer P9-39-46.1
- net VBAT: now also J2.3, J2.4; no longer P9-39-46.3, P9-39-46.4
Changed lines of the file:
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@@
 <part name="S1" library="32bits" deviceset="AS11CH" device="" value="PWR"/>
 <part name="P9-1-10" library="SparkFun-Connectors" deviceset="CONN_05X2" device="PTH" value="bb-pwr"/>
-<part name="P9-39-46" library="SparkFun-Connectors" deviceset="CONN_04X2" device="" value="bb-extra-gnd"/>
-<part name="P8-1-2" library="SparkFun-Connectors" deviceset="CONN_02" device="" value="bb-extra-gnd"/>
 <part name="U6" library="32bits" deviceset="TPS61230A" device=""/>
 <part name="L2" library="Bourns_By_element14_Batch_1" deviceset="PM1210-1R0J-RC" device="" value="1.0 uH"/>
@@
 <part name="R8" library="Vishay_By_element14_Batch_1" deviceset="CRCW08050000Z0EB" device="" value="0Ohm"/>
 <part name="R9" library="32bits" deviceset="NTHS1206N02N1002JE" device="" value="10k"/>
+<part name="U2" library="32bits" deviceset="SI2312BDS-T1-GE3" device=""/>
+<part name="J2" library="32bits" deviceset="2X4-0.01&quot;(2.54MM)-HEADERS" device=""/>
 </parts>
 <sheets>
@@
 <instance part="S1" gate="G$1" x="360.68" y="68.58" rot="R270"/>
 <instance part="P9-1-10" gate="G$1" x="-30.48" y="195.58"/>
-<instance part="P9-39-46" gate="G$1" x="-30.48" y="162.56"/>
-<instance part="P8-1-2" gate="G$1" x="7.62" y="198.12"/>
 <instance part="U6" gate="G$1" x="81.28" y="185.42"/>
 <instance part="L2" gate="A" x="83.82" y="203.2" smashed="yes">
@@
 <instance part="R8" gate="A" x="25.4" y="142.24"/>
 <instance part="R9" gate="G$1" x="355.6" y="152.4" rot="R90"/>
+<instance part="U2" gate="A" x="393.7" y="177.8" rot="R270"/>
+<instance part="J2" gate="A" x="-33.02" y="144.78"/>
 </instances>
 <busses>
 </busses>
 <nets>
-<net name="COPU" class="0">
+<net name="GND" class="0">
 <segment>
 <pinref part="GND1" gate="1" pin="GND"/>
@@
 </segment>
 <segment>
-<pinref part="P8-1-2" gate="G$1" pin="2"/>
-<wire x1="15.24" y1="200.66" x2="22.86" y2="200.66" width="0.1524" layer="91"/>
-<label x="18.796" y="200.914" size="1.778" layer="95"/>
-</segment>
-<segment>
-<pinref part="P8-1-2" gate="G$1" pin="1"/>
-<wire x1="15.24" y1="198.12" x2="22.86" y2="198.12" width="0.1524" layer="91"/>
-<label x="18.796" y="198.374" size="1.778" layer="95"/>
-</segment>
-<segment>
-<pinref part="P9-39-46" gate="G$1" pin="6"/>
-<wire x1="-22.86" y1="162.56" x2="-12.7" y2="162.56" width="0.1524" layer="91"/>
-<label x="-17.272" y="163.068" size="1.778" layer="95"/>
-</segment>
-<segment>
-<pinref part="P9-39-46" gate="G$1" pin="8"/>
-<wire x1="-22.86" y1="160.02" x2="-12.7" y2="160.02" width="0.1524" layer="91"/>
-<label x="-17.272" y="160.274" size="1.778" layer="95"/>
-</segment>
-<segment>
-<pinref part="P9-39-46" gate="G$1" pin="5"/>
-<wire x1="-38.1" y1="162.56" x2="-48.26" y2="162.56" width="0.1524" layer="91"/>
-<label x="-48.006" y="162.814" size="1.778" layer="95"/>
-</segment>
-<segment>
-<pinref part="P9-39-46" gate="G$1" pin="7"/>
-<wire x1="-38.1" y1="160.02" x2="-48.26" y2="160.02" width="0.1524" layer="91"/>
-<label x="-48.006" y="160.274" size="1.778" layer="95"/>
-</segment>
-<segment>
 <pinref part="P8-27-46" gate="G$1" pin="1"/>
 <wire x1="0" y1="182.88" x2="-7.62" y2="182.88" width="0.1524" layer="91"/>
@@
 <wire x1="15.24" y1="144.78" x2="25.4" y2="144.78" width="0.1524" layer="91"/>
 <label x="20.32" y="145.288" size="1.778" layer="95"/>
+</segment>
+<segment>
+<pinref part="J2" gate="A" pin="5"/>
+<wire x1="-38.1" y1="137.16" x2="-48.26" y2="137.16" width="0.1524" layer="91"/>
+</segment>
+<segment>
+<pinref part="J2" gate="A" pin="7"/>
+<wire x1="-38.1" y1="134.62" x2="-48.26" y2="134.62" width="0.1524" layer="91"/>
+</segment>
+<segment>
+<pinref part="J2" gate="A" pin="6"/>
+<wire x1="-22.86" y1="137.16" x2="-15.24" y2="137.16" width="0.1524" layer="91"/>
 </segment>
 </net>
@@
 </segment>
 <segment>
-<pinref part="P9-39-46" gate="G$1" pin="3"/>
-<wire x1="-38.1" y1="165.1" x2="-48.26" y2="165.1" width="0.1524" layer="91"/>
-<label x="-48.006" y="165.354" size="1.778" layer="95"/>
-</segment>
-<segment>
-<pinref part="P9-39-46" gate="G$1" pin="4"/>
-<wire x1="-22.86" y1="165.1" x2="-12.7" y2="165.1" width="0.1524" layer="91"/>
-<label x="-18.796" y="165.608" size="1.778" layer="95"/>
-</segment>
-<segment>
 <pinref part="R8" gate="A" pin="1"/>
 <wire x1="38.1" y1="142.24" x2="48.26" y2="142.24" width="0.1524" layer="91"/>
 <label x="42.164" y="142.748" size="1.778" layer="95"/>
+</segment>
+<segment>
+<pinref part="J2" gate="A" pin="3"/>
+<wire x1="-38.1" y1="139.7" x2="-48.26" y2="139.7" width="0.1524" layer="91"/>
+</segment>
+<segment>
+<pinref part="J2" gate="A" pin="4"/>
+<wire x1="-22.86" y1="139.7" x2="-15.24" y2="139.7" width="0.1524" layer="91"/>
 </segment>
 </net>
@@
 </segment>
 <segment>
-<pinref part="P9-39-46" gate="G$1" pin="1"/>
-<wire x1="-38.1" y1="167.64" x2="-48.26" y2="167.64" width="0.1524" layer="91"/>
-<label x="-53.594" y="167.894" size="1.778" layer="95"/>
+<pinref part="J2" gate="A" pin="1"/>
+<wire x1="-38.1" y1="142.24" x2="-48.26" y2="142.24" width="0.1524" layer="91"/>
 </segment>
 </net>
@@
 </segment>
 </net>
+<net name="N$4" class="0">
+<segment>
+<pinref part="J2" gate="A" pin="8"/>
+<wire x1="-22.86" y1="134.62" x2="-15.24" y2="134.62" width="0.1524" layer="91"/>
+</segment>
+</net>

Commit message: New lithium mechanically complete.
Parts:
- removed P8-27-46: motors, SparkFun-Connectors:CONN_10X2
- removed P9-1-10: bb-pwr, SparkFun-Connectors:CONN_05X2PTH
- removed U2: SI2312BDS-T1-GE3, 32bits:SI2312BDS-T1-GE3
- added J3: motor, 32bits:2X4-0.01"(2.54MM)-JUMPERSSOCKET
- added Q1: (no value), 32bits:SI7137DP
- added R10: 0Ohm, Vishay_By_element14_Batch_1:CRCW08050000Z0EB
- J2: value 2X4-0.01"(2.54MM)-HEADERS -> battery; device 32bits:2X4-0.01"(2.54MM)-HEADERS -> 32bits:2X4-0.01"(2.54MM)-JUMPERSSOCKET
- S1: value PWR -> SS312SAH4; device 32bits:AS11CH -> 32bits:SS312SAH4
Connections:
- removed net N$4: J2.8
- new net THERM_EXT: J2.3, R10.1
- new net VBAT_RAW: J2.1, Q1.DRAIN#5, Q1.DRAIN#6, Q1.DRAIN#7, Q1.DRAIN#8, R8.1
- net GND: now also J3.1, J3.2, J3.3, J3.4, J3.7, J3.8, Q1.GATE; no longer J2.7, P8-27-46.1, P8-27-46.15, P8-27-46.16, P8-27-46.19, P8-27-46.2, P8-27-46.20, P9-1-10.1, P9-1-10.2
- net MOT_6V: now also J3.5, J3.6; no longer P8-27-46.17, P8-27-46.18
- net S1_U4OUT: now also S1.P$1; no longer S1.P$2
- net SYS_5V: now also J2.4; no longer P9-1-10.7, P9-1-10.8
- net U5_THERM: now also R10.2; no longer J2.1
- net VBAT: now also Q1.SOURCE#1, Q1.SOURCE#2, Q1.SOURCE#3; no longer J2.3, J2.4, R8.1
- net VCC: now also S1.P$2; no longer S1.P$1
- net VUSB: now also J2.7; no longer P8-27-46.13, P8-27-46.14
Other:
- moved on the sheet: J1, R8
