File: v3/lithium.sch (EAGLE design)
At the start: 54 parts, among them J1 batt, J2 battery, J3 motor, J4 AVR_ISP, U1 TPS61088VQFN20, U1_C22 8.2nF, U1_CBST 100nF, U1_CCOMP 680PF, U1_CCOMP2 36pF, U1_CIN 0.47uF, U1_CIN2 100nF, U1_COUT 0.47uF, U1_CVCC 1uF, U1_L1 DR73-1R0-R, U1_RCOMP 38.3K Ohms, U1_RFBB 118K Ohms, U1_RFBT 470K Ohms, U1_RLIM 102K Ohms, U1_RT 261K Ohms, U2 ATTINY84-20MU, U4 TPS2113APWR, U4_C3 0.1uF, U4_C4 0.1uF, U4_RPG 100K Ohms, U5 MCP73833-FCI/UN, U5_C1 1.0uF, U5_C2 1.0uF, U5_R1 1K Ohm, U6 TPS61230A, U6_CBST 10 nF, U6_CFF 10pF, U6_CIN 22uF, U6_COUT 22uF, U6_RFBB 100K Ohms, U6_RFBT 316K Ohms

Commit message: Lithium schematic complete.
Parts:
- added D1: 1SS367,H3F, SparkFun-DiscreteSemi:DIODE-SCHOTTKY-BAT20J
- added Q1_R1: 100k, SparkFun-Resistors:100KOHM-0603-1/10W-1%
- added U2_C1, U2_C2: 22uF, 32bits:CAPACITOR0402
- added U2_R1, U2_R2: 10k, SparkFun-Resistors:RESISTOR0402
Connections:
- new net Q1_GATE: D1.A, Q1.GATE, Q1_R1.2
- net GND: now also Q1_R1.1, U2_C1.2, U2_C2.1; no longer Q1.GATE
- net MOSI/SDA: now also U2_R1.1
- net SCK: now also U2_R2.1
- net SYS_5V: now also U2_C1.1, U2_C2.2, U2_R1.2, U2_R2.2
- net VBAT: now also D1.C
Other:
- moved on the sheet: Q1
Changed lines of the file:
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@@
 <part name="J4" library="32bits" deviceset="AVR_ISP" device=""/>
 <part name="U4_RPG" library="Vishay_By_element14_Batch_1" deviceset="CRCW1206100KFKEA" device="" value="100K Ohms"/>
+<part name="U2_C1" library="32bits" deviceset="CAPACITOR" device="0402" value="22uF"/>
+<part name="U2_C2" library="32bits" deviceset="CAPACITOR" device="0402" value="22uF"/>
+<part name="Q1_R1" library="SparkFun-Resistors" deviceset="100KOHM" device="-0603-1/10W-1%" value="100k"/>
+<part name="D1" library="SparkFun-DiscreteSemi" deviceset="DIODE-SCHOTTKY" device="-BAT20J" value="1SS367,H3F"/>
+<part name="U2_R2" library="SparkFun-Resistors" deviceset="RESISTOR" device="0402" value="10k"/>
+<part name="U2_R1" library="SparkFun-Resistors" deviceset="RESISTOR" device="0402" value="10k"/>
 </parts>
 <sheets>
@@
 <instance part="J3" gate="A" x="-7.62" y="195.58"/>
 <instance part="S1" gate="G$1" x="363.22" y="58.42" rot="R90"/>
-<instance part="Q1" gate="G$1" x="17.78" y="233.68"/>
+<instance part="Q1" gate="G$1" x="-7.62" y="251.46"/>
 <instance part="U2" gate="A" x="35.56" y="-38.1"/>
 <instance part="J4" gate="A" x="-12.7" y="213.36"/>
 <instance part="U4_RPG" gate="A" x="292.1" y="53.34" rot="R90"/>
+<instance part="U2_C1" gate="G$1" x="5.08" y="-48.26"/>
+<instance part="U2_C2" gate="G$1" x="5.08" y="-63.5"/>
+<instance part="Q1_R1" gate="G$1" x="-33.02" y="241.3"/>
+<instance part="D1" gate="G$1" x="-22.86" y="233.68" rot="R270"/>
+<instance part="U2_R2" gate="G$1" x="12.7" y="-27.94" rot="R90"/>
+<instance part="U2_R1" gate="G$1" x="236.22" y="-43.18" rot="R90"/>
 </instances>
 <busses>
@@
 </segment>
 <segment>
-<pinref part="Q1" gate="G$1" pin="GATE"/>
-<wire x1="12.7" y1="223.52" x2="2.54" y2="223.52" width="0.1524" layer="91"/>
-<label x="2.794" y="223.774" size="1.778" layer="95"/>
-</segment>
-<segment>
 <pinref part="J3" gate="A" pin="8"/>
 <wire x1="2.54" y1="185.42" x2="10.16" y2="185.42" width="0.1524" layer="91"/>
@@
 <segment>
 <pinref part="U2" gate="A" pin="GND"/>
-<wire x1="38.1" y1="-55.88" x2="22.86" y2="-55.88" width="0.1524" layer="91"/>
 <label x="23.114" y="-55.626" size="1.778" layer="95"/>
+<pinref part="U2_C1" gate="G$1" pin="2"/>
+<wire x1="38.1" y1="-55.88" x2="5.08" y2="-55.88" width="0.1524" layer="91"/>
+<wire x1="5.08" y1="-55.88" x2="5.08" y2="-53.34" width="0.1524" layer="91"/>
+<pinref part="U2_C2" gate="G$1" pin="1"/>
+<wire x1="5.08" y1="-60.96" x2="5.08" y2="-55.88" width="0.1524" layer="91"/>
+<junction x="5.08" y="-55.88"/>
 </segment>
 <segment>
@@
 <wire x1="10.16" y1="205.74" x2="20.32" y2="205.74" width="0.1524" layer="91"/>
 <label x="15.748" y="205.994" size="1.778" layer="95"/>
+</segment>
+<segment>
+<pinref part="Q1_R1" gate="G$1" pin="1"/>
+<wire x1="-38.1" y1="241.3" x2="-48.26" y2="241.3" width="0.1524" layer="91"/>
 </segment>
 </net>
@@
 <pinref part="Q1" gate="G$1" pin="SOURCE#3"/>
 <pinref part="Q1" gate="G$1" pin="SOURCE#2"/>
-<wire x1="12.7" y1="226.06" x2="12.7" y2="228.6" width="0.1524" layer="91"/>
+<wire x1="-12.7" y1="243.84" x2="-12.7" y2="246.38" width="0.1524" layer="91"/>
 <pinref part="Q1" gate="G$1" pin="SOURCE#1"/>
-<wire x1="12.7" y1="228.6" x2="12.7" y2="231.14" width="0.1524" layer="91"/>
-<junction x="12.7" y="228.6"/>
-<wire x1="12.7" y1="231.14" x2="2.54" y2="231.14" width="0.1524" layer="91"/>
-<junction x="12.7" y="231.14"/>
-<label x="2.54" y="231.394" size="1.778" layer="95"/>
+<wire x1="-12.7" y1="246.38" x2="-12.7" y2="248.92" width="0.1524" layer="91"/>
+<junction x="-12.7" y="246.38"/>
+<wire x1="-12.7" y1="248.92" x2="-22.86" y2="248.92" width="0.1524" layer="91"/>
+<junction x="-12.7" y="248.92"/>
+<label x="-22.86" y="249.174" size="1.778" layer="95"/>
 </segment>
 <segment>
@@
 <wire x1="38.1" y1="-48.26" x2="22.86" y2="-48.26" width="0.1524" layer="91"/>
 <label x="22.86" y="-48.006" size="1.778" layer="95"/>
+</segment>
+<segment>
+<pinref part="D1" gate="G$1" pin="C"/>
+<wire x1="-22.86" y1="231.14" x2="-22.86" y2="223.52" width="0.1524" layer="91"/>
+<label x="-23.114" y="220.218" size="1.778" layer="95"/>
 </segment>
 </net>
@@
 <segment>
 <pinref part="U2" gate="A" pin="VCC"/>
-<wire x1="38.1" y1="-58.42" x2="22.86" y2="-58.42" width="0.1524" layer="91"/>
+<wire x1="38.1" y1="-58.42" x2="17.78" y2="-58.42" width="0.1524" layer="91"/>
 <label x="22.86" y="-58.166" size="1.778" layer="95"/>
+<wire x1="17.78" y1="-58.42" x2="17.78" y2="-71.12" width="0.1524" layer="91"/>
+<wire x1="17.78" y1="-71.12" x2="5.08" y2="-71.12" width="0.1524" layer="91"/>
+<pinref part="U2_C2" gate="G$1" pin="2"/>
+<wire x1="5.08" y1="-71.12" x2="5.08" y2="-68.58" width="0.1524" layer="91"/>
 </segment>
 <segment>
 <pinref part="U2" gate="A" pin="(ADC2/AIN1/PCINT2)_PA2"/>
-<wire x1="38.1" y1="-43.18" x2="22.86" y2="-43.18" width="0.1524" layer="91"/>
 <label x="22.86" y="-42.926" size="1.778" layer="95"/>
+<pinref part="U2_C1" gate="G$1" pin="1"/>
+<wire x1="38.1" y1="-43.18" x2="5.08" y2="-43.18" width="0.1524" layer="91"/>
+<wire x1="5.08" y1="-43.18" x2="5.08" y2="-45.72" width="0.1524" layer="91"/>
 </segment>
 <segment>
@@
 <wire x1="10.16" y1="210.82" x2="20.32" y2="210.82" width="0.1524" layer="91"/>
 <label x="15.748" y="211.074" size="1.778" layer="95"/>
+</segment>
+<segment>
+<wire x1="236.22" y1="-38.1" x2="236.22" y2="-30.48" width="0.1524" layer="91"/>
+<label x="232.664" y="-29.718" size="1.778" layer="95"/>
+<pinref part="U2_R1" gate="G$1" pin="2"/>
+</segment>
+<segment>
+<wire x1="12.7" y1="-22.86" x2="12.7" y2="-17.78" width="0.1524" layer="91"/>
+<label x="8.89" y="-17.018" size="1.778" layer="95"/>
+<pinref part="U2_R2" gate="G$1" pin="2"/>
 </segment>
 </net>
@@
 <pinref part="Q1" gate="G$1" pin="DRAIN#5"/>
 <pinref part="Q1" gate="G$1" pin="DRAIN#6"/>
-<wire x1="48.26" y1="223.52" x2="48.26" y2="226.06" width="0.1524" layer="91"/>
+<wire x1="22.86" y1="241.3" x2="22.86" y2="243.84" width="0.1524" layer="91"/>
 <pinref part="Q1" gate="G$1" pin="DRAIN#7"/>
-<wire x1="48.26" y1="226.06" x2="48.26" y2="228.6" width="0.1524" layer="91"/>
-<junction x="48.26" y="226.06"/>
+<wire x1="22.86" y1="243.84" x2="22.86" y2="246.38" width="0.1524" layer="91"/>
+<junction x="22.86" y="243.84"/>
 <pinref part="Q1" gate="G$1" pin="DRAIN#8"/>
-<wire x1="48.26" y1="228.6" x2="48.26" y2="231.14" width="0.1524" layer="91"/>
-<junction x="48.26" y="228.6"/>
-<wire x1="48.26" y1="231.14" x2="58.42" y2="231.14" width="0.1524" layer="91"/>
-<junction x="48.26" y="231.14"/>
-<label x="52.578" y="231.648" size="1.778" layer="95"/>
+<wire x1="22.86" y1="246.38" x2="22.86" y2="248.92" width="0.1524" layer="91"/>
+<junction x="22.86" y="246.38"/>
+<wire x1="22.86" y1="248.92" x2="33.02" y2="248.92" width="0.1524" layer="91"/>
+<junction x="22.86" y="248.92"/>
+<label x="27.178" y="249.428" size="1.778" layer="95"/>
 </segment>
 <segment>
@@
 <segment>
 <pinref part="U2" gate="A" pin="(ADC4/USCK/SCL/T1/PCINT4)_PA4"/>
-<wire x1="38.1" y1="-38.1" x2="22.86" y2="-38.1" width="0.1524" layer="91"/>
+<wire x1="38.1" y1="-38.1" x2="12.7" y2="-38.1" width="0.1524" layer="91"/>
 <label x="22.86" y="-37.846" size="1.778" layer="95"/>
+<wire x1="12.7" y1="-38.1" x2="12.7" y2="-33.02" width="0.1524" layer="91"/>
+<wire x1="12.7" y1="-38.1" x2="2.54" y2="-38.1" width="0.1524" layer="91"/>
+<junction x="12.7" y="-38.1"/>
+<pinref part="U2_R2" gate="G$1" pin="1"/>
 </segment>
 <segment>
@@
 <segment>
 <pinref part="U2" gate="A" pin="PA6"/>
-<wire x1="200.66" y1="-50.8" x2="218.44" y2="-50.8" width="0.1524" layer="91"/>
 <label x="211.328" y="-50.546" size="1.778" layer="95"/>
+<wire x1="200.66" y1="-50.8" x2="236.22" y2="-50.8" width="0.1524" layer="91"/>
+<wire x1="236.22" y1="-50.8" x2="236.22" y2="-48.26" width="0.1524" layer="91"/>
+<wire x1="236.22" y1="-50.8" x2="243.84" y2="-50.8" width="0.1524" layer="91"/>
+<junction x="236.22" y="-50.8"/>
+<pinref part="U2_R1" gate="G$1" pin="1"/>
 </segment>
 <segment>
@@
 </segment>
 </net>
+<net name="Q1_GATE" class="0">
+<segment>
+<pinref part="Q1" gate="G$1" pin="GATE"/>
+<wire x1="-12.7" y1="241.3" x2="-22.86" y2="241.3" width="0.1524" layer="91"/>
+<pinref part="Q1_R1" gate="G$1" pin="2"/>
+<pinref part="D1" gate="G$1" pin="A"/>
+<wire x1="-22.86" y1="241.3" x2="-27.94" y2="241.3" width="0.1524" layer="91"/>
+<wire x1="-22.86" y1="236.22" x2="-22.86" y2="241.3" width="0.1524" layer="91"/>
+<junction x="-22.86" y="241.3"/>
+</segment>
+</net>
