File: v3/lithium.brd (EAGLE design)
At the start: 86.4 x 54.6 mm, 60 parts, among them J1 batt, J2 battery, J3 motor, J4 AVR_ISP, Q1 Si7137DP, Q1_R1 100k, U1 TPS61088VQFN20, U1_C22 8.2nF, U1_CBST 100nF, U1_CCOMP 680PF, U1_CCOMP2 36pF, U1_CIN 0.47uF, U1_CIN2 100nF, U1_COUT 0.47uF, U1_CVCC 1uF, U1_L1 DR73-1R0-R, U1_RCOMP 38.3K Ohms, U1_RFBB 118K Ohms, U1_RFBT 470K Ohms, U1_RLIM 102K Ohms, U1_RT 261K Ohms, U2 ATTINY84-20MU, U2_C1 10nF, U2_C2 2.2uF, U2_R1 10k, U2_R2 10k, U4 TPS2113APWR, U4_C3 0.1uF, U4_C4 0.1uF, U4_RPG 100K Ohms, U5 MCP73833-FCI/UN, U5_C1 1.0uF, U5_C2 1.0uF, U5_R1 1K Ohm, U6 TPS61230A, U6_CBST 10 nF, U6_CFF 10pF, U6_CIN 22uF, U6_COUT 22uF, U6_RFBB 100K Ohms, U6_RFBT 316K Ohms

Commit message: Some cleanup of Lithium layout and repo files.
Parts:
- moved U4_C4 13.6 mm to (74.9, 28.4), turned to 270 degrees
- moved U5_C2 3.79 mm to (73.4, 36.4), turned to 90 degrees
Changed lines of the file:
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@@
 <attribute name="PROD_ID" value="CAP-12417" x="83.6295" y="34.29" size="1.778" layer="27" rot="R270" display="off"/>
 </element>
-<element name="U5_C2" library="SparkFun-Capacitors" package="0402" value="1.0uF" x="71.755" y="39.878" smashed="yes">
-<attribute name="NAME" x="71.755" y="40.64" size="0.254" layer="48" font="vector" ratio="1" align="bottom-center"/>
-<attribute name="PROD_ID" value="CAP-12417" x="71.755" y="39.878" size="1.778" layer="27" display="off"/>
+<element name="U5_C2" library="SparkFun-Capacitors" package="0402" value="1.0uF" x="73.3806" y="36.449" smashed="yes" rot="R90">
+<attribute name="NAME" x="72.6186" y="36.449" size="0.254" layer="48" font="vector" ratio="1" rot="R90" align="bottom-center"/>
+<attribute name="PROD_ID" value="CAP-12417" x="73.3806" y="36.449" size="1.778" layer="27" rot="R90" display="off"/>
 </element>
 <element name="U5_R1" library="Vishay_By_element14_Batch_1" package="RESC1005X40N" value="1K Ohm" x="76.6445" y="39.37" smashed="yes" rot="R90">
@@
 <attribute name="PROD_ID" value="CAP-12416" x="74.0992375" y="31.78591875" size="1.778" layer="27" rot="R45" display="off"/>
 </element>
-<element name="U4_C4" library="SparkFun-Capacitors" package="0402" value="0.1uF" x="71.755" y="41.5925" smashed="yes">
-<attribute name="NAME" x="71.755" y="42.3545" size="0.254" layer="48" font="vector" ratio="1" align="bottom-center"/>
-<attribute name="PROD_ID" value="CAP-12416" x="71.755" y="41.5925" size="1.778" layer="27" display="off"/>
+<element name="U4_C4" library="SparkFun-Capacitors" package="0402" value="0.1uF" x="74.9173" y="28.3718" smashed="yes" rot="R270">
+<attribute name="NAME" x="75.6793" y="28.3718" size="0.254" layer="48" font="vector" ratio="1" rot="R270" align="bottom-center"/>
+<attribute name="PROD_ID" value="CAP-12416" x="74.9173" y="28.3718" size="1.778" layer="27" rot="R270" display="off"/>
 </element>
 <element name="BATT" library="Dialight_By_element14_Batch_1" package="LED_597-3311-407F" value="QTLP650C-4" x="43.815" y="6.35" smashed="yes" rot="R90">
@@
 <via x="74.93" y="16.51" extent="1-16" drill="0.3302"/>
 <via x="70.8152" y="19.1262" extent="1-16" drill="0.3302"/>
-<via x="74.93" y="27.94" extent="1-16" drill="0.3302"/>
 <via x="76.2" y="27.94" extent="1-16" drill="0.3302"/>
+<via x="77.0382" y="27.94" extent="1-16" drill="0.3302"/>
 <via x="80.01" y="21.59" extent="1-16" drill="0.3302"/>
 <via x="79.121" y="30.226" extent="1-16" drill="0.3302"/>
@@
 <via x="86.36" y="40.132" extent="1-16" drill="0.3302"/>
 <via x="83.82" y="45.212" extent="1-16" drill="0.3302"/>
-<via x="72.644" y="38.354" extent="1-16" drill="0.3302"/>
+<via x="75.184" y="40.894" extent="1-16" drill="0.3302"/>
 <via x="81.534" y="39.624" extent="1-16" drill="0.3302"/>
 <via x="80.518" y="40.386" extent="1-16" drill="0.3302"/>
@@
 <contactref element="U4" pad="8"/>
 <contactref element="U4_C4" pad="1"/>
-<wire x1="71.175" y1="41.5925" x2="71.175" y2="39.878" width="0.762" layer="1"/>
 <polygon width="0.2032" layer="1" thermals="no">
 <vertex x="75.7555" y="36.449"/>
@@
 <contactref element="Q1" pad="P$2"/>
 <contactref element="Q1" pad="P$1"/>
-<wire x1="71.175" y1="41.5925" x2="69.922" y2="42.7905" width="0.762" layer="1"/>
-<wire x1="69.922" y1="42.7905" x2="68.58" y2="44.1325" width="0.762" layer="1"/>
 <polygon width="0.2032" layer="1">
 <vertex x="60.9346" y="51.7398"/>
@@
 </polygon>
 <contactref element="U2" pad="5"/>
-<wire x1="71.175" y1="39.878" x2="71.175" y2="37.029" width="0.762" layer="1"/>
-<wire x1="72.39" y1="35.814" x2="71.175" y2="37.029" width="0.762" layer="1"/>
-<wire x1="72.39" y1="35.814" x2="77.1238" y2="35.814" width="0.762" layer="1"/>
 <wire x1="77.1238" y1="35.814" x2="77.1398" y2="35.83" width="0.762" layer="1"/>
 <wire x1="73.6825" y1="29.1875" x2="72.39" y2="30.48" width="0.762" layer="1"/>
-<wire x1="72.39" y1="30.48" x2="72.39" y2="35.814" width="0.762" layer="1"/>
+<wire x1="72.39" y1="35.814" x2="72.39" y2="30.48" width="0.762" layer="1"/>
 <wire x1="76.4511" y1="29.1846" x2="76.454" y2="29.1875" width="0.254" layer="1"/>
 <via x="70.8406" y="20.5994" extent="1-16" drill="0.3302"/>
@@
 <wire x1="58.547" y1="50.4444" x2="60.8203" y2="50.4444" width="0.762" layer="1"/>
 <wire x1="60.8203" y1="50.4444" x2="60.8584" y2="50.4063" width="0.762" layer="1"/>
-<wire x1="68.58" y1="44.1325" x2="59.824221875" y2="44.1325" width="0.762" layer="1"/>
 <wire x1="56.5658" y1="47.1793375" x2="56.5658" y2="48.45815625" width="0.762" layer="1"/>
 <wire x1="58.5654" y1="45.6946" x2="58.404109375" y2="45.6946" width="0.508" layer="1"/>
@@
 <vertex x="76.9874" y="29.0576"/>
 </polygon>
+<wire x1="73.3806" y1="35.869" x2="72.445" y2="35.869" width="0.762" layer="1"/>
+<wire x1="72.445" y1="35.869" x2="72.39" y2="35.814" width="0.762" layer="1" curve="90"/>
+<wire x1="77.1398" y1="35.83" x2="73.4196" y2="35.83" width="0.762" layer="1"/>
+<wire x1="73.4196" y1="35.83" x2="73.3806" y2="35.869" width="0.762" layer="1" curve="-90"/>
+<wire x1="68.6435" y1="44.1325" x2="71.1708" y2="41.6052" width="0.762" layer="1"/>
+<wire x1="71.1708" y1="41.6052" x2="71.1708" y2="37.0332" width="0.762" layer="1"/>
+<wire x1="59.824221875" y1="44.1325" x2="68.6435" y2="44.1325" width="0.762" layer="1"/>
+<wire x1="71.1708" y1="37.0332" x2="72.39" y2="35.814" width="0.762" layer="1"/>
 </signal>
 <signal name="VUSB">
@@
 <wire x1="74.8284" y1="24.43405625" x2="74.8284" y2="24.0792" width="0.1524" layer="16"/>
 <wire x1="81.7048875" y1="25.2984" x2="75.69274375" y2="25.2984" width="0.1524" layer="16"/>
-<wire x1="74.4728" y1="25.88791875" x2="72.7456" y2="27.61511875" width="0.1524" layer="1"/>
+<wire x1="74.4982" y1="25.86251875" x2="72.7456" y2="27.61511875" width="0.1524" layer="1"/>
 <wire x1="72.7456" y1="27.61511875" x2="72.7456" y2="28.8312375" width="0.1524" layer="1"/>
 <wire x1="71.4756" y1="30.1012375" x2="71.4756" y2="33.862775" width="0.1524" layer="1"/>
@@
 <wire x1="70.9295" y1="34.882325" x2="70.9676" y2="34.920425" width="0.1524" layer="1"/>
 <wire x1="70.9676" y1="34.920425" x2="70.9676" y2="35.56" width="0.1524" layer="1"/>
-<wire x1="74.4982" y1="23.7236" x2="74.4728" y2="25.88791875" width="0.1524" layer="1"/>
+<wire x1="74.4982" y1="23.7236" x2="74.4982" y2="25.86251875" width="0.1524" layer="1"/>
 <wire x1="72.7456" y1="28.8312375" x2="71.4756" y2="30.1012375" width="0.1524" layer="1"/>
 <wire x1="71.4756" y1="33.862775" x2="70.9295" y2="34.408875" width="0.1524" layer="1"/>

Commit message: Starting Boron evaluation of bq24160
Parts:
- R7: value 22 Ohms -> 400 Ohms
Changed lines of the file:
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@@
 <attribute name="WATTAGE" value="0.125 W" x="44.45" y="11.4427" size="1.778" layer="27" rot="R90" display="off"/>
 </element>
-<element name="R7" library="Vishay_By_element14_Batch_1" package="RESC1005X40N" value="22 Ohms" x="84.1375" y="31.5595" smashed="yes" rot="R90">
+<element name="R7" library="Vishay_By_element14_Batch_1" package="RESC1005X40N" value="400 Ohms" x="84.1375" y="31.5595" smashed="yes" rot="R90">
 <attribute name="MPN" value="CRCW040222R0JNED" x="84.1375" y="31.5595" size="1.778" layer="27" rot="R90" display="off"/>
 <attribute name="NAME" x="84.8995" y="31.1531" size="0.254" layer="48" ratio="10" rot="SR90"/>

Commit message: Starting Rev 2 of Lithium.
Parts:
- removed D1: 1SS367,H3F, SparkFun-DiscreteSemi:SOD-323
- removed J4: AVR_ISP, 32bits:.1-ISP-PADS
- removed Q1_R1: 100k, SparkFun-Resistors:0603
- removed R7: 400 Ohms, Vishay_By_element14_Batch_1:RESC1005X40N
- removed R9: 10k, 32bits:1206
- removed U2: ATTINY84-20MU, 32bits:20M1
- removed U2_R1: 10k, SparkFun-Resistors:0402
- removed U4: TPS2113APWR, 32bits:PW8
- removed U4_C3, U4_C4: 0.1uF, SparkFun-Capacitors:0402
- removed U4_RPG: 100K Ohms, Vishay_By_element14_Batch_1:RESC3216X71N
- removed U5: MCP73833-FCI/UN, 32bits:MSOP10_MC
- removed U5_C1, U5_C2: 1.0uF, SparkFun-Capacitors:0402
- removed U5_R1: 1K Ohm, Vishay_By_element14_Batch_1:RESC1005X40N
- added J5: FTSH-105-01-XXX-DV-K, FTSH-105-01-XXX-DV-K:FTSH-105-01-XXX-DV-K
- added U3: MKL02Z8VFG4, 32bits:QFN-16_3X3X0.65
- added U7: BQ24168RGET, 32bits:RGE24_2P7X2P7
- moved J1 8.38 mm to (55.1, 48.3), turned to 180 degrees
Connections:
- removed net !RESET: J4.5, U2.13
- removed net MISO: J4.1, U2.20
- removed net Q1_GATE: D1.A, Q1.P$4, Q1_R1.2
- removed net S1_U4OUT: S1.P$1, U4.7
- removed net U4_ILIM: R7.1, U4.4
- removed net U4_STAT: BATT.1, U4.1, U4_RPG.2
- removed net U5_PROG: U5.6, U5_R1.1
- removed net U5_THERM: R9.2, U5.8
- removed net VBAT: D1.C, Q1.P$1, Q1.P$2, Q1.P$3, U2.5, U4.8, U4_C4.1, U5.10, U5.9, U5_C2.1
- new net PGND: U7.17
- new net PGND_2: U7.15
- new net SGND: U7.16
- new net VDDVREFH: U3.1
- new net VREFLVSS: U3.2
- net GND: now also U7.5; no longer J4.6, Q1_R1.1, R7.2, R9.1, U2.8, U4.2, U4.3, U4.5, U4_C3.2, U4_C4.2, U5.5, U5_C1.2, U5_C2.2, U5_R1.2
- net MOSI/SDA: no longer J4.4, U2.16, U2_R1.1
- net MOT_6V: no longer U2.4
- net SCK: now also U3.3; no longer J4.3, U2.1
- net STAT1: no longer U5.3
- net STAT2: no longer U5.4
- net SYS_5V: no longer J4.2, U2.3, U2.9, U2_R1.2
- net U5_NPG: no longer U5.7
- net VBAT_CON: no longer Q1.P$5, Q1.P$6, Q1.P$7, Q1.P$8, Q1.P$9
- net VCC: no longer U4_RPG.1
- net VUSB: no longer U4.6, U4_C3.1, U5.1, U5.2, U5_C1.1
Routing:
- net VBAT: track 52.5 -> 0.00 mm, vias 2 -> 0
- net U4_STAT: track 52.0 -> 0.00 mm, vias 2 -> 0
- net U5_THERM: track 44.8 -> 0.00 mm, vias 2 -> 0
- net VUSB: track 85.7 -> 70.4 mm
- net MISO: track 9.65 -> 0.00 mm, vias 1 -> 0
- net S1_U4OUT: track 8.80 -> 0.00 mm
- net VBAT_CON: track 20.7 -> 12.0 mm
- net !RESET: track 8.28 -> 0.00 mm, vias 1 -> 0
- net VCC: track 65.8 -> 60.3 mm
- net Q1_GATE: track 4.71 -> 0.00 mm
- net MOSI/SDA: track 34.1 -> 30.7 mm
- net SYS_5V: track 130.6 -> 127.4 mm
- net U4_ILIM: track 1.94 -> 0.00 mm
- net VBAT_JST: track 4.45 -> 2.82 mm
- net U5_PROG: track 1.16 -> 0.00 mm
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Other:
- board size 86.4 x 54.6 mm -> 87.6 x 54.6 mm

Commit message: Progress on Lithium rev 2
Connections:
- removed net VREFLVSS: U3.2
- net GND: now also U3.2
